Commit message: add base_footprint frame, fix env variables

File: spot_description/urdf/spot.urdf.xacro (robot description, xacro)
@@ -18,4 +18,10 @@
         <parent link="body" />
         <child link="base_link" />
+    </joint>
+    <link name="base_footprint"/>
+    <joint name="base_footprint_joint" type="fixed">
+        <parent link="base_link"/>
+        <child link="base_footprint"/>
+        <origin xyz="0.0 0.0 -0.5" rpy="0 0 0"/>
     </joint>
     <link name="front_rail"/>
